File: BMS_PCB/Connectors.kicad_sch (KiCad schematic)
At the start: 13 parts, among them J1 Conn_01x37

Commit message: Bohrlöcher
Löcher auf 3,5 mm geändert
Parts:
- H1, H2, H3, H4: footprint MountingHole:MountingHole_3.7mm -> MountingHole:MountingHole_3.5mm
Changed lines of the file:
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@@
 			)
 		)
-		(property "Footprint" "MountingHole:MountingHole_3.7mm"
+		(property "Footprint" "MountingHole:MountingHole_3.5mm"
 			(at 220.98 60.96 0)
 			(effects
@@
 			)
 		)
-		(property "Footprint" "MountingHole:MountingHole_3.7mm"
+		(property "Footprint" "MountingHole:MountingHole_3.5mm"
 			(at 194.31 60.96 0)
 			(effects
@@
 			)
 		)
-		(property "Footprint" "MountingHole:MountingHole_3.7mm"
+		(property "Footprint" "MountingHole:MountingHole_3.5mm"
 			(at 220.98 48.26 0)
 			(effects
@@
 			)
 		)
-		(property "Footprint" "MountingHole:MountingHole_3.7mm"
+		(property "Footprint" "MountingHole:MountingHole_3.5mm"
 			(at 194.31 48.26 0)
 			(effects

Commit message: Bugfix
Capacity und Resistors
Parts:
- C33: footprint Resistor_SMD:R_0603_1608Metric_Pad0.98x0.95mm_HandSolder -> Capacitor_SMD:C_0603_1608Metric_Pad1.08x0.95mm_HandSolder
Changed lines of the file:
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@@
 			)
 		)
-		(property "Footprint" "Resistor_SMD:R_0603_1608Metric_Pad0.98x0.95mm_HandSolder"
+		(property "Footprint" "Capacitor_SMD:C_0603_1608Metric_Pad1.08x0.95mm_HandSolder"
 			(at 75.8952 152.4 0)
 			(effects
